File: sdcard/man/kicad/pocket_power_pack/pocket_power_pack.kicad_sch (KiCad schematic)
At the start: 17 parts, among them J1 SWD_10, SW0 REVERSE, SW1 BRAKE, SW2 FORWARD, SW3 MODE, SW4 F1, SW5 F2, SW6 F3, SW7 POWER

Commit message: Update schematic
Parts:
- removed RAIL1, RAIL2: TestPoint, symbol Connector:TestPoint
- added RAIL1, RAIL2: 2mm socket, symbol Connector_Generic:Conn_01x01
- R1, R2: value 100k -> 22k
- SW1: value BRAKE -> MODE
- SW3: value MODE -> A
- SW4: value F1 -> B
- SW5: value F2 -> C
- SW6: value F3 -> D

Commit message: Update schematics
Parts:
- added C1: C, symbol Device:C
- SW0: value REVERSE -> A REVERSE
- SW1: value MODE -> B MODE
- SW2: value FORWARD -> C FORWARD
- SW3: value A -> D
- SW4: value B -> E
- SW5: value C -> F
- SW6: value D -> G
Connections:
- net GNDD: now also C1.2
Changed lines of the file:
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@@
     (company "spyr.ch")
   )
+  (junction (at 265.43 147.32) (diameter 0) (color 0 0 0 0)
+  )
   (junction (at 187.96 82.55) (diameter 0) (color 0 0 0 0)
   )
+  (junction (at 265.43 154.94) (diameter 0) (color 0 0 0 0)
+  )
   (junction (at 168.91 82.55) (diameter 0) (color 0 0 0 0)
   )
@@
     (stroke (width 0) (type default))
   )
-  (wire (pts (xy 248.92 148.59) (xy 265.43 148.59))
+  (wire (pts (xy 248.92 147.32) (xy 265.43 147.32))
     (stroke (width 0) (type default))
   )
@@
     (stroke (width 0) (type default))
   )
-  (wire (pts (xy 265.43 87.63) (xy 265.43 148.59))
+  (wire (pts (xy 265.43 87.63) (xy 265.43 147.32))
     (stroke (width 0) (type default))
   )
@@
     (stroke (width 0) (type default))
   )
-  (wire (pts (xy 265.43 156.21) (xy 265.43 154.94))
+  (wire (pts (xy 265.43 160.02) (xy 265.43 154.94))
     (stroke (width 0) (type default))
   )
@@
     )
   )
+  (symbol (lib_id "Device:C") (at 265.43 151.13 0) (unit 1)
+    (in_bom yes) (on_board yes) (dnp no) (fields_autoplaced)
+    (property "Reference" "C1" (at 269.24 149.86 0)
+      (effects (font (size 1.27 1.27)) (justify left))
+    )
+    (property "Value" "C" (at 269.24 152.4 0)
+      (effects (font (size 1.27 1.27)) (justify left))
+    )
+    (property "Footprint" "" (at 266.3952 154.94 0)
+      (effects (font (size 1.27 1.27)) hide)
+    )
+    (property "Datasheet" "~" (at 265.43 151.13 0)
+      (effects (font (size 1.27 1.27)) hide)
+    )
+    (pin "2")
+    (pin "1")
+    (instances
+      (project "pocket_power_pack"
+        (path "/9538e4ed-27e6-4c37-b989-9859dc0d49e8"
+          (reference "C1") (unit 1)
+        )
+      )
+    )
+  )
   (symbol (lib_id "Device:R") (at 168.91 116.84 0) (unit 1)
     (in_bom yes) (on_board yes) (dnp no) (fields_autoplaced)
@@
       (effects (font (size 1.27 1.27)) (justify left))
     )
-    (property "Value" "C" (at 144.78 168.91 90)
+    (property "Value" "F" (at 144.78 168.91 90)
       (effects (font (size 1.27 1.27)) (justify left))
     )
@@
       (effects (font (size 1.27 1.27)) (justify left))
     )
-    (property "Value" "B" (at 130.81 168.91 90)
+    (property "Value" "E" (at 130.81 168.91 90)
       (effects (font (size 1.27 1.27)) (justify left))
     )
@@
       (effects (font (size 1.27 1.27)) (justify left))
     )
-    (property "Value" "MODE" (at 137.16 143.51 90)
+    (property "Value" "B MODE" (at 137.16 143.51 90)
       (effects (font (size 1.27 1.27)) (justify left))
     )
@@
     )
   )
-  (symbol (lib_id "power:GNDD") (at 265.43 156.21 0) (unit 1)
+  (symbol (lib_id "power:GNDD") (at 265.43 160.02 0) (unit 1)
     (in_bom yes) (on_board yes) (dnp no) (fields_autoplaced)
-    (property "Reference" "#PWR07" (at 265.43 162.56 0)
+    (property "Reference" "#PWR07" (at 265.43 166.37 0)
       (effects (font (size 1.27 1.27)) hide)
     )
-    (property "Value" "GNDD" (at 265.43 161.29 0)
+    (property "Value" "GNDD" (at 265.43 165.1 0)
       (effects (font (size 1.27 1.27)))
     )
-    (property "Footprint" "" (at 265.43 156.21 0)
+    (property "Footprint" "" (at 265.43 160.02 0)
       (effects (font (size 1.27 1.27)) hide)
     )
-    (property "Datasheet" "" (at 265.43 156.21 0)
+    (property "Datasheet" "" (at 265.43 160.02 0)
       (effects (font (size 1.27 1.27)) hide)
     )
@@
       (effects (font (size 1.27 1.27)) (justify left))
     )
-    (property "Value" "A" (at 116.84 168.91 90)
+    (property "Value" "D" (at 116.84 168.91 90)
       (effects (font (size 1.27 1.27)) (justify left))
     )
@@
       (effects (font (size 1.27 1.27)) (justify left))
     )
-    (property "Value" "D" (at 158.75 168.91 90)
+    (property "Value" "G" (at 158.75 168.91 90)
       (effects (font (size 1.27 1.27)) (justify left))
     )
@@
       (effects (font (size 1.27 1.27)) (justify left))
     )
-    (property "Value" "FORWARD" (at 151.13 143.51 90)
+    (property "Value" "C FORWARD" (at 151.13 143.51 90)
       (effects (font (size 1.27 1.27)) (justify left))
     )
@@
       (effects (font (size 1.27 1.27)) (justify left))
     )
-    (property "Value" "REVERSE" (at 123.19 143.51 90)
+    (property "Value" "A REVERSE" (at 123.19 143.51 90)
       (effects (font (size 1.27 1.27)) (justify left))
     )
